Commit message: feat(helios_description): add mesh models, update URDF geometry

File: src/helios_description/urdf/base.xacro (robot description, xacro)
@@ -11,8 +11,24 @@
   <xacro:property name="half_wheelbase" value="0.110"/>   <!-- wheelbase 0.220 / 2 (front<->rear) -->
   <xacro:property name="half_track"     value="0.165"/>   <!-- track 0.330 / 2 (left<->right) -->
-  <!-- Chassis body box (rough; A4WD3 frame ~ 0.32 x 0.24 x 0.10). -->
+  <!-- Chassis collision box (rough; A4WD3 frame ~ 0.32 x 0.24 x 0.10). Kept as a
+       primitive per meshes/README.md even though visual now uses the CAD mesh. -->
   <xacro:property name="chassis_length" value="0.320"/>
   <xacro:property name="chassis_width"  value="0.240"/>
   <xacro:property name="chassis_height" value="0.0785"/>
+  <!-- CAD meshes (meshes/*.STL) were exported in millimeters with a Y-up,
+       Z-forward convention (verified consistently across chassis/wheel/lidar/
+       zed bounding boxes: mesh_y -> robot up, mesh_z -> robot forward,
+       mesh_x -> robot left). mesh_scale converts mm -> m; mesh_rpy is the
+       fixed rotation that maps the CAD frame into REP-103 (x fwd, y left,
+       z up). mesh_*_xyz below re-center each mesh's bounding-box centroid on
+       its link origin (computed from the STL bounding boxes, not measured).
+       TODO: this is a best-effort derivation from bbox dimensions matching
+       known hardware specs — confirm visually in RViz and nudge if a mesh
+       looks rotated/flipped. -->
+  <xacro:property name="mesh_scale" value="0.001 0.001 0.001"/>
+  <xacro:property name="mesh_rpy"   value="${pi/2} 0 ${pi/2}"/>
+  <xacro:property name="chassis_mesh_xyz" value="-0.16552 -0.13383 -0.03827"/>
+  <xacro:property name="wheelA_mesh_xyz"  value="-0.08398 -0.02833 -0.08436"/>
+  <xacro:property name="wheelB_mesh_xyz"  value="-0.08395 -0.02833 -0.08436"/>
   <!-- ===================== Materials ===================== -->
   <material name="chassis_grey"><color rgba="0.30 0.32 0.35 1.0"/></material>
@@ -22,7 +38,7 @@
   <link name="base_link">
     <visual>
-      <origin xyz="0 0 0" rpy="0 0 0"/>
+      <origin xyz="${chassis_mesh_xyz}" rpy="${mesh_rpy}"/>
       <geometry>
-        <box size="${chassis_length} ${chassis_width} ${chassis_height}"/>
+        <mesh filename="package://helios_description/meshes/Rover-Chassis.STL" scale="${mesh_scale}"/>
       </geometry>
       <material name="chassis_grey"/>
@@ -49,10 +65,17 @@
   </joint>
   <!-- ===================== Wheel macro ===================== -->
-  <xacro:macro name="wheel" params="name x y">
+  <!-- mesh_file/mesh_xyz select one of the two A4WD3 mecanum wheel meshes.
+       Mecanum wheels are handed: rollers on diagonal corners mirror each
+       other so the X-roller pattern lets the drivetrain strafe. Assigned
+       here as the standard diagonal pairing (A: front_left/rear_right,
+       B: front_right/rear_left) — TODO: verify against the A4WD3 assembly
+       manual / look at the physical rover and swap mesh_file per-corner
+       below if the rollers look mirrored in RViz. -->
+  <xacro:macro name="wheel" params="name x y mesh_file mesh_xyz">
     <link name="${name}_wheel">
       <visual>
-        <origin xyz="0 0 0" rpy="${pi/2} 0 0"/>
+        <origin xyz="${mesh_xyz}" rpy="${mesh_rpy}"/>
         <geometry>
-          <cylinder radius="${wheel_radius}" length="${wheel_width}"/>
+          <mesh filename="package://helios_description/meshes/${mesh_file}" scale="${mesh_scale}"/>
         </geometry>
         <material name="wheel_black"/>
@@ -78,7 +101,11 @@
   </xacro:macro>
   <!-- Corner names match the wheel_odometry node. -->
-  <xacro:wheel name="front_left"  x="${half_wheelbase}"  y="${half_track}"/>
-  <xacro:wheel name="front_right" x="${half_wheelbase}"  y="${-half_track}"/>
-  <xacro:wheel name="rear_left"   x="${-half_wheelbase}" y="${half_track}"/>
-  <xacro:wheel name="rear_right"  x="${-half_wheelbase}" y="${-half_track}"/>
+  <xacro:wheel name="front_left"  x="${half_wheelbase}"  y="${half_track}"
+               mesh_file="A4WD3-W-ME-A.STL" mesh_xyz="${wheelA_mesh_xyz}"/>
+  <xacro:wheel name="front_right" x="${half_wheelbase}"  y="${-half_track}"
+               mesh_file="A4WD3-W-ME-B.STL" mesh_xyz="${wheelB_mesh_xyz}"/>
+  <xacro:wheel name="rear_left"   x="${-half_wheelbase}" y="${half_track}"
+               mesh_file="A4WD3-W-ME-B.STL" mesh_xyz="${wheelB_mesh_xyz}"/>
+  <xacro:wheel name="rear_right"  x="${-half_wheelbase}" y="${-half_track}"
+               mesh_file="A4WD3-W-ME-A.STL" mesh_xyz="${wheelA_mesh_xyz}"/>
 </robot>

File: src/helios_description/urdf/sensors.xacro (robot description, xacro)
@@ -15,10 +15,19 @@
   <link name="zed_camera_link">
     <visual>
+      <!-- mesh_rpy/mesh_scale from base.xacro (shared CAD-frame convention).
+           TODO: verify visually — camera may need yaw += pi if it's facing
+           backwards (mesh forward-axis sign was inferred, not measured). -->
+      <origin xyz="-0.02128 -0.08888 -0.01547" rpy="${mesh_rpy}"/>
+      <geometry>
+        <mesh filename="package://helios_description/meshes/ZED2i.STL" scale="${mesh_scale}"/>
+      </geometry>
+      <material name="sensor_blue"/>
+    </visual>
+    <collision>
       <origin xyz="0 0 0" rpy="0 0 0"/>
       <geometry>
         <box size="0.04 0.180 0.030"/>   <!-- ZED 2i ~175 mm wide -->
       </geometry>
-      <material name="sensor_blue"/>
-    </visual>
+    </collision>
   </link>
   <joint name="zed_mount_joint" type="fixed">
@@ -32,10 +41,16 @@
   <link name="laser">
     <visual>
+      <origin xyz="-0.03163 -0.02500 -0.03500" rpy="${mesh_rpy}"/>
+      <geometry>
+        <mesh filename="package://helios_description/meshes/Hokuyo-UST-10LX-Lidar.STL" scale="${mesh_scale}"/>
+      </geometry>
+      <material name="sensor_blue"/>
+    </visual>
+    <collision>
       <origin xyz="0 0 0" rpy="0 0 0"/>
       <geometry>
         <cylinder radius="0.020" length="0.0685"/>   <!-- UST-10LX ~50 mm dia -->
       </geometry>
-      <material name="sensor_blue"/>
-    </visual>
+    </collision>
   </link>
   <joint name="laser_mount_joint" type="fixed">

Commit message: fix(helios_description): correct sensor mount positions in URDF

File: src/helios_description/urdf/base.xacro (robot description, xacro)
@@ -11,19 +11,15 @@
   <xacro:property name="half_wheelbase" value="0.110"/>   <!-- wheelbase 0.220 / 2 (front<->rear) -->
   <xacro:property name="half_track"     value="0.165"/>   <!-- track 0.330 / 2 (left<->right) -->
-  <!-- Chassis collision box (rough; A4WD3 frame ~ 0.32 x 0.24 x 0.10). Kept as a
-       primitive per meshes/README.md even though visual now uses the CAD mesh. -->
+  <!-- Chassis collision box (rough; A4WD3 frame ~ 0.32 x 0.24 x 0.10). -->
   <xacro:property name="chassis_length" value="0.320"/>
   <xacro:property name="chassis_width"  value="0.240"/>
   <xacro:property name="chassis_height" value="0.0785"/>
-  <!-- CAD meshes (meshes/*.STL) were exported in millimeters with a Y-up,
-       Z-forward convention (verified consistently across chassis/wheel/lidar/
-       zed bounding boxes: mesh_y -> robot up, mesh_z -> robot forward,
+  <!-- CAD meshes (meshes/*.STL) were exported in millimeters with a Y-up,Z-forward convention
+      zed bounding boxes: mesh_y -> robot up, mesh_z -> robot forward,
        mesh_x -> robot left). mesh_scale converts mm -> m; mesh_rpy is the
        fixed rotation that maps the CAD frame into REP-103 (x fwd, y left,
        z up). mesh_*_xyz below re-center each mesh's bounding-box centroid on
-       its link origin (computed from the STL bounding boxes, not measured).
-       TODO: this is a best-effort derivation from bbox dimensions matching
-       known hardware specs — confirm visually in RViz and nudge if a mesh
-       looks rotated/flipped. -->
+       its link origin.
+       -->
   <xacro:property name="mesh_scale" value="0.001 0.001 0.001"/>
   <xacro:property name="mesh_rpy"   value="${pi/2} 0 ${pi/2}"/>
@@ -67,9 +63,5 @@
   <!-- mesh_file/mesh_xyz select one of the two A4WD3 mecanum wheel meshes.
        Mecanum wheels are handed: rollers on diagonal corners mirror each
-       other so the X-roller pattern lets the drivetrain strafe. Assigned
-       here as the standard diagonal pairing (A: front_left/rear_right,
-       B: front_right/rear_left) — TODO: verify against the A4WD3 assembly
-       manual / look at the physical rover and swap mesh_file per-corner
-       below if the rollers look mirrored in RViz. -->
+       other so the X-roller pattern lets the drivetrain strafe.-->
   <xacro:macro name="wheel" params="name x y mesh_file mesh_xyz">
     <link name="${name}_wheel">
@@ -102,10 +94,10 @@
   <!-- Corner names match the wheel_odometry node. -->
   <xacro:wheel name="front_left"  x="${half_wheelbase}"  y="${half_track}"
-               mesh_file="A4WD3-W-ME-A.STL" mesh_xyz="${wheelA_mesh_xyz}"/>
+               mesh_file="A4WD3-W-ME-B.STL" mesh_xyz="${wheelA_mesh_xyz}"/>
   <xacro:wheel name="front_right" x="${half_wheelbase}"  y="${-half_track}"
-               mesh_file="A4WD3-W-ME-B.STL" mesh_xyz="${wheelB_mesh_xyz}"/>
+               mesh_file="A4WD3-W-ME-A.STL" mesh_xyz="${wheelB_mesh_xyz}"/>
   <xacro:wheel name="rear_left"   x="${-half_wheelbase}" y="${half_track}"
-               mesh_file="A4WD3-W-ME-B.STL" mesh_xyz="${wheelB_mesh_xyz}"/>
+               mesh_file="A4WD3-W-ME-A.STL" mesh_xyz="${wheelB_mesh_xyz}"/>
   <xacro:wheel name="rear_right"  x="${-half_wheelbase}" y="${-half_track}"
-               mesh_file="A4WD3-W-ME-A.STL" mesh_xyz="${wheelA_mesh_xyz}"/>
+               mesh_file="A4WD3-W-ME-B.STL" mesh_xyz="${wheelA_mesh_xyz}"/>
 </robot>

File: src/helios_description/urdf/sensors.xacro (robot description, xacro)
@@ -2,20 +2,19 @@
 <!--
   Sensor mount frames: ZED 2i camera and Hokuyo UST-10LX LiDAR.
-  ALL origins below are ROUGH PLACEHOLDERS. Measure the real mount offsets from
-  the rover center (base_link) on your CAD / rover and update the <origin> of
-  each *_mount_joint. xyz in meters, rpy in radians (REP-103: x fwd, y left, z up).
+  Frame convention REP-103: x forward, y left, z up. base_link at the rover
+  geometric center, at wheel-axle height. The ZED wrapper's root camera frame
+  is zed_camera_link, which is attached to the rover via a fixed joint. The
+  Hokuyo's frame is named 'laser' to match urg_node2's frame_id, so /scan lands here. Both sensors mount on the top surface of the chassis box.
 -->
 <robot xmlns:xacro="http://www.ros.org/wiki/xacro">
   <!-- ===================== ZED 2i ===================== -->
   <!-- 'zed_camera_link' is the ZED wrapper's root camera frame. This joint
-       attaches it to the rover. NOTE: make sure the ZED wrapper is NOT also
-       publishing a base_link -> zed_camera_link transform (otherwise the frame
-       gets two parents). In the wrapper config set publish_tf so it only
+       attaches it to the rover.
+       NOTE: make sure the ZED wrapper is NOT also publishing a base_link -> zed_camera_link transform
+       (otherwise the frame gets two parents). In the wrapper config set publish_tf so it only
        publishes the camera's *internal* frames, and let this URDF own the mount. -->
   <link name="zed_camera_link">
     <visual>
-      <!-- mesh_rpy/mesh_scale from base.xacro (shared CAD-frame convention).
-           TODO: verify visually — camera may need yaw += pi if it's facing
-           backwards (mesh forward-axis sign was inferred, not measured). -->
+      <!-- mesh_rpy/mesh_scale from base.xacro (shared CAD-frame convention). -->
       <origin xyz="-0.02128 -0.08888 -0.01547" rpy="${mesh_rpy}"/>
       <geometry>
@@ -34,6 +33,6 @@
     <parent link="base_link"/>
     <child link="zed_camera_link"/>
-    <!-- TODO: measure. Placeholder: front edge, raised. -->
-    <origin xyz="0.140 0.0 0.03925" rpy="0 0 0"/>
+    <!-- Placeholder: top plate, leading edge, centerline. -->
+    <origin xyz="0.101 0.0 0.050" rpy="0 -1.5708 0"/>
   </joint>
   <!-- ===================== Hokuyo UST-10LX ===================== -->
@@ -57,6 +56,6 @@
     <parent link="base_link"/>
     <child link="laser"/>
-    <!-- TODO: measure. Placeholder: front-center, on top. -->
-    <origin xyz="0.140 0.0 0.07925" rpy="0 0 0"/>
+    <!-- Placeholder: top plate, aft of the ZED. -->
+    <origin xyz="0.045 0 0.100" rpy="0 0 0"/>
   </joint>
 </robot>

Commit message: fix(helios_description): move chassis inertial link to base_link_inertia, adjust sensor mountings for the new top plate

File: src/helios_description/urdf/base.xacro (robot description, xacro)
@@ -46,4 +46,9 @@
       </geometry>
     </collision>
+  </link>
+  <!-- base_link_inertia: KDL doesn't support inertia on the root link, so the
+       chassis mass lives here instead (fixed, identity offset from base_link)
+       rather than on base_link itself. -->
+  <link name="base_link_inertia">
     <inertial>
       <mass value="5.0"/>
@@ -52,4 +57,9 @@
     </inertial>
   </link>
+  <joint name="base_link_inertia_joint" type="fixed">
+    <parent link="base_link"/>
+    <child link="base_link_inertia"/>
+    <origin xyz="0 0 0" rpy="0 0 0"/>
+  </joint>
   <!-- base_footprint: ground projection below base_link (child, so base_link
        keeps a single parent = odom from the odometry node). -->

File: src/helios_description/urdf/sensors.xacro (robot description, xacro)
@@ -37,5 +37,5 @@
     <child link="zed_camera_link"/>
     <!-- Placeholder: top plate, leading edge, centerline. -->
-    <origin xyz="0.101 0.0 0.050" rpy="0 0 0"/>
+    <origin xyz="0.106 0.0 0.050" rpy="0 0 0"/>
   </joint>
   <!-- ===================== Hokuyo UST-10LX ===================== -->
@@ -60,5 +60,5 @@
     <child link="laser"/>
     <!-- Placeholder: top plate, aft of the ZED. -->
-    <origin xyz="0.045 0 0.100" rpy="0 0 0"/>
+    <origin xyz="0.05 0 0.100" rpy="0 0 0"/>
   </joint>
 </robot>

Commit message: refactor(helios_description): move shared mesh props and materials to common.xacro and fixed sensor mountin points to measured values. sensors.xacro consumed mesh_scale/mesh_rpy and the materials without defining them. Included once from the top level. Joints were placeholder. replaced with measured values.

File: src/helios_description/urdf/base.xacro (robot description, xacro)
@@ -15,20 +15,11 @@
   <xacro:property name="chassis_width"  value="0.240"/>
   <xacro:property name="chassis_height" value="0.0785"/>
-  <!-- CAD meshes (meshes/*.STL) were exported in millimeters with a Y-up,Z-forward convention
-      zed bounding boxes: mesh_y -> robot up, mesh_z -> robot forward,
-       mesh_x -> robot left). mesh_scale converts mm -> m; mesh_rpy is the
-       fixed rotation that maps the CAD frame into REP-103 (x fwd, y left,
-       z up). mesh_*_xyz below re-center each mesh's bounding-box centroid on
-       its link origin.
-       -->
-  <xacro:property name="mesh_scale" value="0.001 0.001 0.001"/>
-  <xacro:property name="mesh_rpy"   value="${pi/2} 0 ${pi/2}"/>
+  <!-- mesh_scale, mesh_rpy and the materials live in common.xacro, which
+       helios.urdf.xacro includes before this file. The mesh_*_xyz values
+       below re-center each mesh's bounding-box centroid on its link origin
+       and are specific to these meshes, so they stay here. -->
   <xacro:property name="chassis_mesh_xyz" value="-0.16552 -0.13383 -0.03827"/>
   <xacro:property name="wheelA_mesh_xyz"  value="-0.08398 -0.02833 -0.08436"/>
   <xacro:property name="wheelB_mesh_xyz"  value="-0.08395 -0.02833 -0.08436"/>
-  <!-- ===================== Materials ===================== -->
-  <material name="chassis_grey"><color rgba="0.30 0.32 0.35 1.0"/></material>
-  <material name="wheel_black"><color rgba="0.10 0.10 0.10 1.0"/></material>
-  <material name="sensor_blue"><color rgba="0.10 0.30 0.80 1.0"/></material>
   <!-- ===================== base_link (root) ===================== -->
   <link name="base_link">

File: src/helios_description/urdf/helios.urdf.xacro (robot description, xacro)
@@ -2,8 +2,12 @@
 <!--
   Helios rover (Lynxmotion A4WD3 Mecanum) — top-level xacro.
-  Composes base.xacro (chassis + wheels) and
-  sensors.xacro (ZED + LiDAR mount frames).
+  Composes common.xacro (shared properties + materials),
+  base.xacro (chassis + wheels) and sensors.xacro (ZED + LiDAR mount frames).
+  common.xacro MUST come first — the other two consume its properties and
+  materials. base.xacro and sensors.xacro are independent of each other and
+  may be listed in either order.
 -->
 <robot name="helios" xmlns:xacro="http://www.ros.org/wiki/xacro">
+  <xacro:include filename="$(find helios_description)/urdf/common.xacro"/>
   <xacro:include filename="$(find helios_description)/urdf/base.xacro"/>
   <xacro:include filename="$(find helios_description)/urdf/sensors.xacro"/>

File: src/helios_description/urdf/sensors.xacro (robot description, xacro)
@@ -7,4 +7,12 @@
   Hokuyo's frame is named 'laser' to match urg_node2's frame_id, so /scan lands here.
   Both sensors mount on the top surface of the chassis box.
+  Consumes mesh_scale and the sensor_blue material from common.xacro, which
+  helios.urdf.xacro includes before this file.
+  MOUNT ACCURACY: these joint origins are the ONLY source of the
+  base_link -> sensor transforms — both drivers run publish_tf:=false, so
+  nothing else corrects them. The EKF uses zed_mount_joint to rotate ZED VIO
+  twist into base_link, and slam_toolbox uses laser_mount_joint as the
+  scan-matching lever arm. A wrong number here is a silent accuracy bug, not
+  a rendering glitch. Per-joint status is noted at each joint below.
 -->
 <robot xmlns:xacro="http://www.ros.org/wiki/xacro">
@@ -36,5 +44,18 @@
     <parent link="base_link"/>
     <child link="zed_camera_link"/>
-    <!-- Placeholder: top plate, leading edge, centerline. -->
+    <!-- Top plate, leading edge, centerline. MEASURED by hand against the real
+         rover.
+         Measured to the point the ZED wrapper actually anchors to: its
+         zed_camera_link is the threaded screw hole in the BOTTOM face of the
+         camera ("Camera mounting point" in the wrapper's zed_macro.urdf.xacro),
+         not the lens and not the body centre. The wrapper hangs
+         zed_camera_center 15 mm above it and the left lens a further -10 mm x /
+         +60 mm y off that.
+         rpy VERIFIED: the ZED is physically mounted flat and forward-facing.
+         (An earlier -90/+90 pitch here was compensating for the mesh's own CAD
+         axes, not real geometry, and was corrupting how the EKF rotated ZED
+         velocity into base_link.)
+         z of 0.050 sits 11 mm above the top plate (surface is at ~0.039);
+         that is the mount standoff, not an error. -->
     <origin xyz="0.106 0.0 0.050" rpy="0 0 0"/>
   </joint>
@@ -59,5 +80,15 @@
     <parent link="base_link"/>
     <child link="laser"/>
-    <!-- Placeholder: top plate, aft of the ZED. -->
+    <!-- Top plate, aft of the ZED. MEASURED by hand against the real rover.
+         slam_toolbox uses this offset as its scan-matching lever arm: an error
+         of d here becomes a prediction error of (R(phi) - I)*d, i.e. up to 2*d
+         on a 180 deg turn, which is why it is worth measuring rather than
+         estimating. xyz is to the laser's optical centre (the rotating mirror
+         inside the case, not the base of the housing).
+         rpy is 0 0 0, which asserts the Hokuyo's 0 deg bearing points straight
+         forward, i.e. the cable and the 90 deg dead zone face AFT. If the
+         sensor is ever remounted cable-forward this must become 0 0 ${pi};
+         nothing downstream would report an error, the map would just be built
+         backwards. -->
     <origin xyz="0.05 0 0.100" rpy="0 0 0"/>
   </joint>
